File: Design/energy_harvesting.sch (KiCad schematic (older format))
At the start: 5 parts, among them U2 74LVC1G3157

Commit message: Improvement over the Power management: - added TPS6201DRC for raising leaking voltage from supercapacitor - supercap is protected from overvoltage using a shunt diode - power management is using MOSFET logic (2 PFET, 1 NFET)
Parts:
- removed D5: ZPD3.3, Diode_THT:D_DO-35_SOD27_P10.16mm_Horizontal, symbol Diode:ZPDxx
- removed U2: 74LVC1G3157, symbol 74xGxx:74LVC1G3157
- added C1, C2, C3: 10mF, symbol Device:C
- added C4: 2uF, symbol Device:C
- added D2: 220mV, symbol Device:D_Schottky
- added L2: 2.2uH, symbol Device:L
- added Q1: Q_NMOS_DGS, symbol Device:Q_NMOS_DGS
- added Q2, Q3: Q_PMOS_DSG, symbol Device:Q_PMOS_DSG
- added R1: 4M3, symbol Device:R
- added R2: 6M2, symbol Device:R
- added U1: TLV431DCK, Package_TO_SOT_SMD:SOT-363_SC-70-6, symbol Reference_Voltage:TL431DCK
- added U2: TPS61201DRC, Package_SON:Texas_S-PVSON-N10_ThermalVias, symbol Regulator_Switching:TPS61201DRC
- EDLC1: renamed from Super_Cap1; footprint (none) -> Connector_PinHeader_1.27mm:PinHeader_1x02_P1.27mm_Vertical
- L1: renamed from L4; value 1uH -> MMZ2012S121AT000; symbol Device:L -> Device:L_Core_Ferrite
Connections:
- net GND: now also EDLC1.1, C1.2, C2.1, C3.1, C4.2, R2.1, U1.6 (A), U2.11 (PAD), U2.4 (PGND), U2.9 (GND); no longer EDLC1.2
- net VDD: now also C3.2, Q1.3 (S), Q3.2 (S); no longer L1.2
- net at D1.1 (+): now also L1.1, C1.1, Q1.2 (G), Q2.3 (G), Q3.3 (G); no longer EDLC1.1
- net NFC1 renamed Energy_NFC_1
- net NFC2 renamed Energy_NFC_2
- new net: C2.2, D2.1 (K), EDLC1.2, Q1.1 (D), Q2.1 (D), R1.2, U1.1 (K)
- new net: D2.2 (A), L1.2
- new net: C4.1, U2.1 (VAUX)
- new net: Q3.1 (D), U2.10 (FB), U2.2 (VOUT)
- new net: L2.2, U2.3 (L)
- new net: L2.1, Q2.2 (S), U2.5 (VIN), U2.6 (EN), U2.7 (UVLO), U2.8 (PS)
- new net: R1.1, R2.2, U1.3 (REF)
Other:
- note added: "490mV"
- note added: "630mV"
- note added: "Energy harvesting"
- moved on the sheet: D1, EDLC1

Commit message: - designed configurable intensity for RGB LEDs - included Breakout (FET, Diode, etc.) Spice models from Cadence Spice - replaced global label with hierarchical complete view - customized net labels with pin function - exported first spice netlist which presents small bugs
Parts:
- removed D2: 220mV, symbol Device:D_Schottky
- removed Q2: Q_PMOS_DSG, symbol Device:Q_PMOS_DSG
- added Q1: Q_NMOS_DGS, symbol Device:Q_NMOS_DGS
- added Q2: Q_DUAL_NMOS_G1S2G2D2S1D1, symbol Device:Q_DUAL_NMOS_G1S2G2D2S1D1
- added R1: 1k, symbol Device:R
- added R2, R6, R7: 10M, symbol Device:R
- added R3: 2880m, symbol Device:R
- added V1: VSOURCE, symbol pspice:VSOURCE
- C1, C2, C3: Spice_Model (none) -> 10m; Spice_Netlist_Enabled (none) -> Y; Spice_Primitive (none) -> C
- C4: Spice_Model (none) -> 2u; Spice_Netlist_Enabled (none) -> Y; Spice_Primitive (none) -> C
- EDLC1: Spice_Model (none) -> 1; Spice_Netlist_Enabled (none) -> Y; Spice_Primitive (none) -> C
- L1: Spice_Lib_File (none) -> C:\\Users\\steve.huguenin\\Documents\\PSPICE\\Librairies PS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; Spice_Model (none) -> MMZ2012S121AT000_s; Spice_Netlist_Enabled (none) -> Y; Spice_Node_Sequence (none) -> 5.40000000E-07; Spice_Primitive (none) -> X
- L2: Spice_Model (none) -> 2.2u; Spice_Netlist_Enabled (none) -> Y; Spice_Primitive (none) -> L
- Q3: renamed from Q1; Spice_Lib_File (none) -> C:\\Cadence\\SPB_17.2\\tools\\pspice\\library\\breakout.lib; Spice_Model (none) -> MBreakND; Spice_Netlist_Enabled (none) -> Y; Spice_Primitive (none) -> M
- Q4: renamed from Q3; value Q_PMOS_DSG -> Q_NMOS_DGS; symbol Device:Q_PMOS_DSG -> Device:Q_NMOS_DGS; Spice_Lib_File (none) -> C:\\Cadence\\SPB_17.2\\tools\\pspice\\library\\breakout.lib; Spice_Model (none) -> MBreakND; Spice_Netlist_Enabled (none) -> Y; Spice_Primitive (none) -> M
- R4: renamed from R1; Spice_Model (none) -> 4Meg3; Spice_Netlist_Enabled (none) -> Y; Spice_Primitive (none) -> R
- R5: renamed from R2; Spice_Model (none) -> 6Meg2; Spice_Netlist_Enabled (none) -> Y; Spice_Primitive (none) -> R
- U1: Spice_Lib_File (none) -> C:\\Users\\steve.huguenin\\Documents\\PSPICE\\Librairies PS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; Spice_Model (none) -> TLV431; Spice_Netlist_Enabled (none) -> Y; Spice_Primitive (none) -> X
- U2: Spice_Lib_File (none) -> C:\\Users\\steve.huguenin\\Documents\\PSPICE\\Librairies PS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; Spice_Model (none) -> TPS61220_TRANS; Spice_Netlist_Enabled (none) -> N; Spice_Primitive (none) -> X
Connections:
- net VDD: now also Q4.1 (D); no longer Q4.2 (S)
- net at EDLC1.2, R4.2, U1.1 (K): now also Q1.3 (S), Q2.6 (D), R3.2; no longer C2.2, Q3.1 (D)
- net V1: now reaches C1.1, D1.1 (+), L1.1
- net V1: now also V1.1 (E1); no longer Q3.2 (G), Q4.3 (G)
- net at L1.2: now also C2.2, Q3.1 (D), Q2.1 (G), R1.2, R6.2
- net at U2.10 (FB), U2.2 (VOUT): now also Q4.3 (S), R7.2; no longer Q4.1 (D)
- net at L2.1, U2.5 (VIN), U2.6 (EN)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: now also Q2.3 (G), Q2.4 (D), Q2.5 (S)
- net GND renamed 0
- net 0: now also Q2.2 (S), R3.1, V1.2 (E2)
- new net: Q1.1 (D), R1.1, R2.2
- new net: Q1.2 (G), R2.1
- new net: Q3.2 (G), R6.1
- new net: Q4.2 (G), R7.1
Other:
- note added: "-140mV"
- note removed: "140mV"
- moved on the sheet: C1, C2, C3, C4, EDLC1, L1, L2, Q3, Q4, R4, R5, U1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
